Commit message: Adjust the urdf model

File: src/yahboomcar_description/urdf/yahboomcar_M1_gazebo.urdf.xacro (robot description, xacro)
@@ -3,6 +3,10 @@
      Commit Version: 1.6.0-4-g7f85cfe  Build Version: 1.6.7995.38578
      For more information, please see http://wiki.ros.org/sw_urdf_exporter -->
-<robot name="yahboomcar_M1" xmlns:xacro="http://ros.org/wiki/xacro">
+<robot name="yahboomcar_M1"
+       xmlns:xacro="http://ros.org/wiki/xacro"
+       xmlns:ignition="http://ignitionrobotics.org/schema">
   <xacro:arg name="enable_gpu_lidar" default="true"/>
+  <xacro:arg name="enable_contact_sensors" default="false"/>
+  <xacro:arg name="enable_force_torque_sensors" default="false"/>
   <link name="imu_link"/>
   <link
@@ -76,7 +80,5 @@
     </visual>
     <collision>
-      <origin
-        xyz="0 0 0"
-        rpy="1.5708 0 0" />
+      <origin xyz="0 0 0" rpy="1.5708 0 0" />
       <geometry>
         <cylinder radius="0.04" length="0.035"/>
@@ -88,5 +90,5 @@
     type="continuous">
     <origin
-      xyz="0.092963 0.08425 0.012478"
+      xyz="0.093 0.08425 0.0125"
       rpy="0 0 0" />
     <parent
@@ -131,7 +133,5 @@
     </visual>
     <collision>
-      <origin
-        xyz="0 0 0"
-        rpy="1.5708 0 0" />
+      <origin xyz="0 0 0" rpy="1.5708 0 0" />
       <geometry>
         <cylinder radius="0.04" length="0.035"/>
@@ -143,5 +143,5 @@
     type="continuous">
     <origin
-      xyz="-0.093021 0.08425 0.012513"
+      xyz="-0.093 0.08425 0.0125"
       rpy="0 0 0" />
     <parent
@@ -186,7 +186,5 @@
     </visual>
     <collision>
-      <origin
-        xyz="0 0 0"
-        rpy="1.5708 0 0" />
+      <origin xyz="0 0 0" rpy="1.5708 0 0" />
       <geometry>
         <cylinder radius="0.04" length="0.035"/>
@@ -198,5 +196,5 @@
     type="continuous">
     <origin
-      xyz="0.092979 -0.08425 0.012487"
+      xyz="0.093 -0.08425 0.0125"
       rpy="0 0 0" />
     <parent
@@ -241,7 +239,5 @@
     </visual>
     <collision>
-      <origin
-        xyz="0 0 0"
-        rpy="1.5708 0 0" />
+      <origin xyz="0 0 0" rpy="1.5708 0 0" />
       <geometry>
         <cylinder radius="0.04" length="0.035"/>
@@ -253,5 +249,5 @@
     type="continuous">
     <origin
-      xyz="-0.092963 -0.08425 0.012478"
+      xyz="-0.093 -0.08425 0.0125"
       rpy="0 0 0" />
     <parent
@@ -384,5 +380,8 @@
     <parent link="base_footprint"/>
     <child link="base_link"/>
-    <origin xyz="0.0 0.0 0.0215" rpy="0 0 0"/>
+    <!-- Put base_footprint at the wheel-ground contact plane.  The wheel
+         centers are about 0.0125 m above base_link and the wheels have a
+         0.04 m radius. -->
+    <origin xyz="0.0 0.0 0.0275" rpy="0 0 0"/>
   </joint>
   <!-- Gazebo Sim extensions for the M1 model.  The mesh geometry and joint
@@ -390,23 +389,143 @@
        added here. -->
   <gazebo reference="le_fr_Link">
-    <mu1>1.0</mu1>
-    <mu2>0.0</mu2>
-    <fdir1>1 -1 0</fdir1>
+    <collision>
+      <surface>
+        <friction>
+          <ode>
+            <mu>1.0</mu>
+            <mu2>0.1</mu2>
+            <fdir1 ignition:expressed_in="base_footprint">1 -1 0</fdir1>
+          </ode>
+        </friction>
+      </surface>
+    </collision>
+    <xacro:if value="$(arg enable_contact_sensors)">
+      <sensor name="le_fr_contact" type="contact">
+        <always_on>true</always_on>
+        <update_rate>100</update_rate>
+        <contact>
+          <collision>le_fr_Link_collision</collision>
+          <topic>/m1/contact/le_fr</topic>
+        </contact>
+      </sensor>
+    </xacro:if>
   </gazebo>
+  <xacro:if value="$(arg enable_force_torque_sensors)">
+    <gazebo reference="le_fr_joint">
+      <sensor name="le_fr_force_torque" type="force_torque">
+        <always_on>true</always_on>
+        <update_rate>100</update_rate>
+        <force_torque>
+          <frame>parent</frame>
+          <measure_direction>child_to_parent</measure_direction>
+        </force_torque>
+      </sensor>
+    </gazebo>
+  </xacro:if>
   <gazebo reference="le_be_Link">
-    <mu1>1.0</mu1>
-    <mu2>0.0</mu2>
-    <fdir1>1 1 0</fdir1>
+    <collision>
+      <surface>
+        <friction>
+          <ode>
+            <mu>1.0</mu>
+            <mu2>0.1</mu2>
+            <fdir1 ignition:expressed_in="base_footprint">1 1 0</fdir1>
+          </ode>
+        </friction>
+      </surface>
+    </collision>
+    <xacro:if value="$(arg enable_contact_sensors)">
+      <sensor name="le_be_contact" type="contact">
+        <always_on>true</always_on>
+        <update_rate>100</update_rate>
+        <contact>
+          <collision>le_be_Link_collision</collision>
+          <topic>/m1/contact/le_be</topic>
+        </contact>
+      </sensor>
+    </xacro:if>
   </gazebo>
+  <xacro:if value="$(arg enable_force_torque_sensors)">
+    <gazebo reference="le_be_joint">
+      <sensor name="le_be_force_torque" type="force_torque">
+        <always_on>true</always_on>
+        <update_rate>100</update_rate>
+        <force_torque>
+          <frame>parent</frame>
+          <measure_direction>child_to_parent</measure_direction>
+        </force_torque>
+      </sensor>
+    </gazebo>
+  </xacro:if>
   <gazebo reference="ri_fr_Link">
-    <mu1>1.0</mu1>
-    <mu2>0.0</mu2>
-    <fdir1>1 1 0</fdir1>
+    <collision>
+      <surface>
+        <friction>
+          <ode>
+            <mu>1.0</mu>
+            <mu2>0.1</mu2>
+            <fdir1 ignition:expressed_in="base_footprint">1 1 0</fdir1>
+          </ode>
+        </friction>
+      </surface>
+    </collision>
+    <xacro:if value="$(arg enable_contact_sensors)">
+      <sensor name="ri_fr_contact" type="contact">
+        <always_on>true</always_on>
+        <update_rate>100</update_rate>
+        <contact>
+          <collision>ri_fr_Link_collision</collision>
+          <topic>/m1/contact/ri_fr</topic>
+        </contact>
+      </sensor>
+    </xacro:if>
   </gazebo>
+  <xacro:if value="$(arg enable_force_torque_sensors)">
+    <gazebo reference="ri_fr_joint">
+      <sensor name="ri_fr_force_torque" type="force_torque">
+        <always_on>true</always_on>
+        <update_rate>100</update_rate>
+        <force_torque>
+          <frame>parent</frame>
+          <measure_direction>child_to_parent</measure_direction>
+        </force_torque>
+      </sensor>
+    </gazebo>
+  </xacro:if>
   <gazebo reference="ri_be_Link">
-    <mu1>1.0</mu1>
-    <mu2>0.0</mu2>
-    <fdir1>1 -1 0</fdir1>
+    <collision>
+      <surface>
+        <friction>
+          <ode>
+            <mu>1.0</mu>
+            <mu2>0.1</mu2>
+            <fdir1 ignition:expressed_in="base_footprint">1 -1 0</fdir1>
+          </ode>
+        </friction>
+      </surface>
+    </collision>
+    <xacro:if value="$(arg enable_contact_sensors)">
+      <sensor name="ri_be_contact" type="contact">
+        <always_on>true</always_on>
+        <update_rate>100</update_rate>
+        <contact>
+          <collision>ri_be_Link_collision</collision>
+          <topic>/m1/contact/ri_be</topic>
+        </contact>
+      </sensor>
+    </xacro:if>
   </gazebo>
+  <xacro:if value="$(arg enable_force_torque_sensors)">
+    <gazebo reference="ri_be_joint">
+      <sensor name="ri_be_force_torque" type="force_torque">
+        <always_on>true</always_on>
+        <update_rate>100</update_rate>
+        <force_torque>
+          <frame>parent</frame>
+          <measure_direction>child_to_parent</measure_direction>
+        </force_torque>
+      </sensor>
+    </gazebo>
+  </xacro:if>
   <xacro:if value="$(arg enable_gpu_lidar)">
     <!-- T-MINI PLUS profile: 0.54 deg angular resolution, 12 Hz, 0.05 to 12 m. -->
@@ -453,5 +572,5 @@
       <wheel_radius>0.04</wheel_radius>
       <topic>/cmd_vel</topic>
-      <odom_topic>/odom</odom_topic>
+      <odom_topic>/wheel_odom</odom_topic>
       <min_acceleration>-1.0</min_acceleration>
       <max_acceleration>1.0</max_acceleration>
@@ -460,6 +579,6 @@
             name="ignition::gazebo::systems::OdometryPublisher">
       <odom_frame>odom</odom_frame>
-      <robot_base_frame>base_link</robot_base_frame>
-      <child_frame_id>base_link</child_frame_id>
+      <robot_base_frame>base_footprint</robot_base_frame>
+      <child_frame_id>base_footprint</child_frame_id>
       <odom_publish_frequency>30</odom_publish_frequency>
       <odom_topic>/odom</odom_topic>

Commit message: fix(sim): use dual Ogre GPU LiDAR scans

File: src/yahboomcar_description/urdf/yahboomcar_M1_gazebo.urdf.xacro (robot description, xacro)
@@ -7,4 +7,5 @@
        xmlns:ignition="http://ignitionrobotics.org/schema">
   <xacro:arg name="enable_gpu_lidar" default="true"/>
+  <xacro:arg name="dual_gpu_lidar" default="true"/>
   <xacro:arg name="gpu_lidar_min_angle" default="-3.14159265359"/>
   <xacro:arg name="gpu_lidar_max_angle" default="3.14159265359"/>
@@ -373,4 +374,21 @@
       velocity="1000" />
   </joint>
+  <!-- Keep the exported housing frame separate from the LiDAR measurement
+       frame.  The STL bounds place laser_Link's origin near the physical
+       optical-window height, so the initial measurement offset is zero. -->
+  <link name="laser_scan_link"/>
+  <joint name="laser_scan_joint" type="fixed">
+    <parent link="laser_Link"/>
+    <child link="laser_scan_link"/>
+    <origin xyz="0 0 0" rpy="0 0 0"/>
+  </joint>
+  <xacro:if value="$(arg dual_gpu_lidar)">
+    <link name="laser_scan_rear_link"/>
+    <joint name="laser_scan_rear_joint" type="fixed">
+      <parent link="laser_scan_link"/>
+      <child link="laser_scan_rear_link"/>
+      <origin xyz="0 0 0" rpy="0 0 3.14159265359"/>
+    </joint>
+  </xacro:if>
   <joint name="base_imu" type="fixed">
   <parent link="base_link"/>
@@ -533,35 +551,100 @@
   </xacro:if>
   <xacro:if value="$(arg enable_gpu_lidar)">
-    <!-- T-MINI PLUS profile: 0.54 deg angular resolution, 12 Hz, 0.05 to 12 m. -->
-    <gazebo reference="laser_Link">
-      <sensor name="tmini_plus" type="gpu_lidar">
-        <topic>/scan</topic>
-        <update_rate>12</update_rate>
-        <always_on>true</always_on>
-        <visualize>false</visualize>
-        <ray>
-          <scan>
-            <horizontal>
-              <samples>667</samples>
-              <resolution>1</resolution>
-              <min_angle>$(arg gpu_lidar_min_angle)</min_angle>
-              <max_angle>$(arg gpu_lidar_max_angle)</max_angle>
-            </horizontal>
-            <vertical>
-              <samples>1</samples>
-              <resolution>1</resolution>
-              <min_angle>0</min_angle>
-              <max_angle>0</max_angle>
-            </vertical>
-          </scan>
-          <range>
-            <min>0.05</min>
-            <max>12.0</max>
-            <resolution>0.01</resolution>
-          </range>
-        </ray>
-        <gz_frame_id>laser_Link</gz_frame_id>
-      </sensor>
-    </gazebo>
+    <!-- Keep the historical single-360 sensor as the positive-control path. -->
+    <xacro:unless value="$(arg dual_gpu_lidar)">
+      <gazebo reference="laser_scan_link">
+        <sensor name="tmini_plus" type="gpu_lidar">
+          <topic>/scan</topic>
+          <update_rate>12</update_rate>
+          <always_on>true</always_on>
+          <visualize>false</visualize>
+          <ray>
+            <scan>
+              <horizontal>
+                <samples>667</samples>
+                <resolution>1</resolution>
+                <min_angle>$(arg gpu_lidar_min_angle)</min_angle>
+                <max_angle>$(arg gpu_lidar_max_angle)</max_angle>
+              </horizontal>
+              <vertical>
+                <samples>1</samples>
+                <resolution>1</resolution>
+                <min_angle>0</min_angle>
+                <max_angle>0</max_angle>
+              </vertical>
+            </scan>
+            <range>
+              <min>0.05</min>
+              <max>12.0</max>
+              <resolution>0.01</resolution>
+            </range>
+          </ray>
+          <gz_frame_id>laser_scan_link</gz_frame_id>
+        </sensor>
+      </gazebo>
+    </xacro:unless>
+    <!-- Ogre1 renders two coincident half scans; TF rotates the rear scan. -->
+    <xacro:if value="$(arg dual_gpu_lidar)">
+      <gazebo reference="laser_scan_link">
+        <sensor name="tmini_plus_front" type="gpu_lidar">
+          <topic>/scan_front</topic>
+          <update_rate>12</update_rate>
+          <always_on>true</always_on>
+          <visualize>false</visualize>
+          <ray>
+            <scan>
+              <horizontal>
+                <samples>334</samples>
+                <resolution>1</resolution>
+                <min_angle>-1.57079632679</min_angle>
+                <max_angle>1.57079632679</max_angle>
+              </horizontal>
+              <vertical>
+                <samples>1</samples>
+                <resolution>1</resolution>
+                <min_angle>0</min_angle>
+                <max_angle>0</max_angle>
+              </vertical>
+            </scan>
+            <range>
+              <min>0.05</min>
+              <max>12.0</max>
+              <resolution>0.01</resolution>
+            </range>
+          </ray>
+          <gz_frame_id>laser_scan_link</gz_frame_id>
+        </sensor>
+      </gazebo>
+      <gazebo reference="laser_scan_rear_link">
+        <sensor name="tmini_plus_rear" type="gpu_lidar">
+          <topic>/scan_rear</topic>
+          <update_rate>12</update_rate>
+          <always_on>true</always_on>
+          <visualize>false</visualize>
+          <ray>
+            <scan>
+              <horizontal>
+                <samples>334</samples>
+                <resolution>1</resolution>
+                <min_angle>-1.57079632679</min_angle>
+                <max_angle>1.57079632679</max_angle>
+              </horizontal>
+              <vertical>
+                <samples>1</samples>
+                <resolution>1</resolution>
+                <min_angle>0</min_angle>
+                <max_angle>0</max_angle>
+              </vertical>
+            </scan>
+            <range>
+              <min>0.05</min>
+              <max>12.0</max>
+              <resolution>0.01</resolution>
+            </range>
+          </ray>
+          <gz_frame_id>laser_scan_rear_link</gz_frame_id>
+        </sensor>
+      </gazebo>
+    </xacro:if>
   </xacro:if>
   <gazebo>
